File: pcb/Feather.sch (KiCad schematic (older format))
At the start: 34 parts, among them J1 MicroUSB, J2 JST Connector, J3 ANT, J4 U.FL, J5 Conn_01x03, J6 Conn_01x12, J7 Conn_01x16, SW1 KMR2, U1 ATSAMD21G18A-M, U2 AP2112K-3.3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

Commit message: Se crea la biblioteca Adafruit_PinHeader para las tiras de pines que se deben soldar en los costados de la placa. Con esta modificación, se actualizo también el circuito esquemático. Listo para corregir y avanzar con el desarrollo del PCB.
Parts:
- J3: footprint Connector_Pin:Pin_D1.0mm_L10.0mm -> Adafruit_PinHeader_2.54mm:Adafruit_Feather_PinHeader_1x01_P2.54mm
- J5: footprint Connector_PinHeader_2.54mm:PinHeader_1x03_P2.54mm_Vertical -> Adafruit_PinHeader_2.54mm:Adafruit_Feather_PinHeader_1x03_P2.54mm
- J6: footprint Connector_PinHeader_2.54mm:PinHeader_1x12_P2.54mm_Vertical -> Adafruit_PinHeader_2.54mm:Adafruit_Feather_PinHeader_1x12_P2.54mm
- J7: footprint Connector_PinHeader_2.54mm:PinHeader_1x16_P2.54mm_Vertical -> Adafruit_PinHeader_2.54mm:Adafruit_Feather_PinHeader_1x16_P2.54mm
Changed lines of the file:
@@
 F 0 "J3" H 10320 3402 50  0000 L CNN
 F 1 "ANT" H 10320 3311 50  0000 L CNN
-F 2 "Connector_Pin:Pin_D1.0mm_L10.0mm" H 10240 3360 50  0001 C CNN
+F 2 "Adafruit_PinHeader_2.54mm:Adafruit_Feather_PinHeader_1x01_P2.54mm" H 10240 3360 50  0001 C CNN
 F 3 "~" H 10240 3360 50  0001 C CNN
 	1    10240 3360
@@
 F 0 "J5" H 5995 3720 50  0000 L CNN
 F 1 "Conn_01x03" H 6120 3461 50  0001 L CNN
-F 2 "Connector_PinHeader_2.54mm:PinHeader_1x03_P2.54mm_Vertical" H 6040 3510 50  0001 C CNN
+F 2 "Adafruit_PinHeader_2.54mm:Adafruit_Feather_PinHeader_1x03_P2.54mm" H 6040 3510 50  0001 C CNN
 F 3 "~" H 6040 3510 50  0001 C CNN
 	1    6040 3510
@@
 F 0 "J6" H 5990 5175 50  0000 L CNN
 F 1 "Conn_01x12" H 6115 4461 50  0001 L CNN
-F 2 "Connector_PinHeader_2.54mm:PinHeader_1x12_P2.54mm_Vertical" H 6035 4560 50  0001 C CNN
+F 2 "Adafruit_PinHeader_2.54mm:Adafruit_Feather_PinHeader_1x12_P2.54mm" H 6035 4560 50  0001 C CNN
 F 3 "~" H 6035 4560 50  0001 C CNN
 	1    6035 4560
@@
 F 0 "J7" H 5990 7145 50  0000 L CNN
 F 1 "Conn_01x16" H 6115 6231 50  0001 L CNN
-F 2 "Connector_PinHeader_2.54mm:PinHeader_1x16_P2.54mm_Vertical" H 6035 6330 50  0001 C CNN
+F 2 "Adafruit_PinHeader_2.54mm:Adafruit_Feather_PinHeader_1x16_P2.54mm" H 6035 6330 50  0001 C CNN
 F 3 "~" H 6035 6330 50  0001 C CNN
 	1    6035 6330

Commit message: Se realizan leves ajustes en el esquemático y se adiciona el archivo de licencia. Listo para revisar.
Parts:
- added FID1: Fiducial, Fiducial:Fiducial_0.5mm_Mask1mm, symbol Mechanical:Fiducial
- added H1, H3: Mounting Hole w/Pad, MountingHole:MountingHole_2.5mm_Pad, symbol Mechanical:MountingHole_Pad
- added H2, H4: Mounting Hole, MountingHole:MountingHole_2.5mm, symbol Mechanical:MountingHole
- J1: value MicroUSB -> 10118192
- J2: value JST Connector -> S2B-PH-SM4-TB
- J4: value U.FL -> U.FL-R-SMT-1
Connections:
- no-connect marks 11 -> 13
Other:
- note added: "1) All resistors are 0603 size.\n\n2) All capacitors except for C6, C8, C9 and C10 are 0603 size.\n\n3) Capcitors C6, C8, C9 and C10 are 0805 size.\n\n4) All LEDs are 0805 size."
- note added: "4 X M2.5 Screws"
- note added: "CPU"
- note added: "Mounting Holes & Fiducials"
- note added: "Reset"
- note removed: "1) All resistors are 0603 size.\n\n2) All capacitors except for C6, C8, C9 and C10 are 0603 size.\n\n3) Capcitors C6, C8, C9 and C10 are 0805 size.\n\n1) All LEDs are 0805 size."
- note removed: "CPU & Reset"
- moved on the sheet: C1, C2, C3, C4, J5, J6, J7, SW1, TP1, TP2, U1, Y1
