File: pcb/Feather.sch (KiCad schematic (older format))
At the start: 39 parts, among them J1 10118192, J2 S2B-PH-SM4-TB, J3 ANT, J4 U.FL-R-SMT-1, J5 Conn_01x03, J6 Conn_01x12, J7 Conn_01x16, SW1 KMR2, U1 ATSAMD21G18A-M, U2 AP2112K-3.3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

Commit message: Se modifica todo el proyecto para utilizar componentes 0805 en lugar de 0603 que se usan en el circuito original. Se incorpora archivo del PCB, con componentes posicionados y con modelos 3D incluídos.
Parts:
- C1, C2, C3, C4, C7: footprint Capacitor_SMD:C_0603_1608Metric -> Capacitor_SMD:C_0805_2012Metric
- C5: value 1uF -> 10uF; footprint Capacitor_SMD:C_0603_1608Metric -> Capacitor_SMD:C_0805_2012Metric
- FID1: footprint Fiducial:Fiducial_0.5mm_Mask1mm -> Fiducial:Fiducial_1mm_Mask2mm
- H1, H3: footprint MountingHole:MountingHole_2.5mm_Pad -> Adafruit:MountingHole_2.5mm_Pad_TopOnly
- H2, H4: footprint MountingHole:MountingHole_2.5mm -> Adafruit:MountingHole_2.5mm
- J2: footprint Connector_JST:JST_ACH_BM02B-ACHSS-GAN-ETF_1x02-1MP_P1.20mm_Vertical -> Connector_JST:JST_PH_S2B-PH-SM4-TB_1x02-1MP_P2.00mm_Horizontal
- J3: footprint Adafruit_PinHeader_2.54mm:Adafruit_Feather_PinHeader_1x01_P2.54mm -> Adafruit:Adafruit_Feather_PinHeader_1x01_P2.54mm
- J5: footprint Adafruit_PinHeader_2.54mm:Adafruit_Feather_PinHeader_1x03_P2.54mm -> Adafruit:Adafruit_Feather_PinHeader_1x03_P2.54mm
- J6: footprint Adafruit_PinHeader_2.54mm:Adafruit_Feather_PinHeader_1x12_P2.54mm -> Adafruit:Adafruit_Feather_PinHeader_1x12_P2.54mm
- J7: footprint Adafruit_PinHeader_2.54mm:Adafruit_Feather_PinHeader_1x16_P2.54mm -> Adafruit:Adafruit_Feather_PinHeader_1x16_P2.54mm
- R1, R3, R4, R5, R6, R7: footprint Resistor_SMD:R_0603_1608Metric -> Resistor_SMD:R_0805_2012Metric
Other:
- note added: "1) Originally, all resistors were 0603. For this project, they were all changed to 0805.\n\n2) Capacitors C5, C6, C8, C9 and C10 are 0805 size.\n\n3) Originally, capacitors C1, C2, C3, C4 and C7 were 0603 size. \nFor this project, they were all changed to 0805.\n\n4) All LEDs are 0805 size for better visibility."
- note removed: "1) All resistors are 0603 size.\n\n2) All capacitors except for C6, C8, C9 and C10 are 0603 size.\n\n3) Capcitors C6, C8, C9 and C10 are 0805 size.\n\n4) All LEDs are 0805 size."
Changed lines of the file:
@@
 F 0 "C1" V 2415 3165 50  0000 R CNN
 F 1 "1uF" V 2670 3205 50  0000 R CNN
-F 2 "Capacitor_SMD:C_0603_1608Metric" H 2550 3135 50  0001 C CNN
+F 2 "Capacitor_SMD:C_0805_2012Metric" H 2550 3135 50  0001 C CNN
 F 3 "~" H 2550 3135 50  0001 C CNN
 	1    2550 3135
@@
 F 0 "C2" H 1060 4380 50  0000 C CNN
 F 1 "22pF" H 1100 4290 50  0000 C CNN
-F 2 "Capacitor_SMD:C_0603_1608Metric" H 915 4330 50  0001 C CNN
+F 2 "Capacitor_SMD:C_0805_2012Metric" H 915 4330 50  0001 C CNN
 F 3 "~" H 915 4330 50  0001 C CNN
 	1    915  4330
@@
 F 0 "C4" H 1618 4284 50  0000 R CNN
 F 1 "1uF" H 1618 4375 50  0000 R CNN
-F 2 "Capacitor_SMD:C_0603_1608Metric" H 1710 4330 50  0001 C CNN
+F 2 "Capacitor_SMD:C_0805_2012Metric" H 1710 4330 50  0001 C CNN
 F 3 "~" H 1710 4330 50  0001 C CNN
 	1    1710 4330
@@
 F 0 "C3" H 1580 4380 50  0000 C CNN
 F 1 "22pF" H 1620 4290 50  0000 C CNN
-F 2 "Capacitor_SMD:C_0603_1608Metric" H 1435 4330 50  0001 C CNN
+F 2 "Capacitor_SMD:C_0805_2012Metric" H 1435 4330 50  0001 C CNN
 F 3 "~" H 1435 4330 50  0001 C CNN
 	1    1435 4330
@@
 F 0 "R1" V 1545 1450 50  0000 C CNN
 F 1 "100k" V 1620 1450 50  0000 C CNN
-F 2 "Resistor_SMD:R_0603_1608Metric" H 1465 1450 50  0001 C CNN
+F 2 "Resistor_SMD:R_0805_2012Metric" H 1465 1450 50  0001 C CNN
 F 3 "~" H 1465 1450 50  0001 C CNN
 	1    1465 1450
@@
 P 1080 1655
 F 0 "C5" H 988 1701 50  0000 R CNN
-F 1 "1uF" H 988 1610 50  0000 R CNN
-F 2 "Capacitor_SMD:C_0603_1608Metric" H 1080 1655 50  0001 C CNN
+F 1 "10uF" H 988 1610 50  0000 R CNN
+F 2 "Capacitor_SMD:C_0805_2012Metric" H 1080 1655 50  0001 C CNN
 F 3 "~" H 1080 1655 50  0001 C CNN
 	1    1080 1655
@@
 F 0 "C7" H 2723 1701 50  0000 R CNN
 F 1 "1uF" H 2723 1610 50  0000 R CNN
-F 2 "Capacitor_SMD:C_0603_1608Metric" H 2815 1655 50  0001 C CNN
+F 2 "Capacitor_SMD:C_0805_2012Metric" H 2815 1655 50  0001 C CNN
 F 3 "~" H 2815 1655 50  0001 C CNN
 	1    2815 1655
@@
 F 0 "J2" H 5650 1445 50  0000 L CNN
 F 1 "S2B-PH-SM4-TB" H 5425 1125 50  0000 L CNN
-F 2 "Connector_JST:JST_ACH_BM02B-ACHSS-GAN-ETF_1x02-1MP_P1.20mm_Vertical" H 5695 1335 50  0001 C CNN
+F 2 "Connector_JST:JST_PH_S2B-PH-SM4-TB_1x02-1MP_P2.00mm_Horizontal" H 5695 1335 50  0001 C CNN
 F 3 "https://www.jst-mfg.com/product/pdf/eng/ePH.pdf" H 5695 1335 50  0001 C CNN
 	1    5695 1335
@@
 F 0 "R3" V 7975 1120 50  0000 C CNN
 F 1 "1k" V 8155 1120 50  0000 C CNN
-F 2 "Resistor_SMD:R_0603_1608Metric" H 8065 1120 50  0001 C CNN
+F 2 "Resistor_SMD:R_0805_2012Metric" H 8065 1120 50  0001 C CNN
 F 3 "~" H 8065 1120 50  0001 C CNN
 	1    8065 1120
@@
 F 0 "R4" V 6890 1575 50  0000 C CNN
 F 1 "10k" V 7070 1575 50  0000 C CNN
-F 2 "Resistor_SMD:R_0603_1608Metric" H 6980 1575 50  0001 C CNN
+F 2 "Resistor_SMD:R_0805_2012Metric" H 6980 1575 50  0001 C CNN
 F 3 "~" H 6980 1575 50  0001 C CNN
 	1    6980 1575
@@
 F 0 "R5" H 9384 1306 50  0000 L CNN
 F 1 "100k" H 9384 1215 50  0000 L CNN
-F 2 "Resistor_SMD:R_0603_1608Metric" H 9325 1260 50  0001 C CNN
+F 2 "Resistor_SMD:R_0805_2012Metric" H 9325 1260 50  0001 C CNN
 F 3 "~" H 9325 1260 50  0001 C CNN
 	1    9325 1260
@@
 F 0 "J3" H 10320 3402 50  0000 L CNN
 F 1 "ANT" H 10320 3311 50  0000 L CNN
-F 2 "Adafruit_PinHeader_2.54mm:Adafruit_Feather_PinHeader_1x01_P2.54mm" H 10240 3360 50  0001 C CNN
+F 2 "Adafruit:Adafruit_Feather_PinHeader_1x01_P2.54mm" H 10240 3360 50  0001 C CNN
 F 3 "~" H 10240 3360 50  0001 C CNN
 	1    10240 3360
@@
 F 0 "J5" H 5460 3420 50  0000 L CNN
 F 1 "Conn_01x03" H 5585 3161 50  0001 L CNN
-F 2 "Adafruit_PinHeader_2.54mm:Adafruit_Feather_PinHeader_1x03_P2.54mm" H 5505 3210 50  0001 C CNN
+F 2 "Adafruit:Adafruit_Feather_PinHeader_1x03_P2.54mm" H 5505 3210 50  0001 C CNN
 F 3 "~" H 5505 3210 50  0001 C CNN
 	1    5505 3210
@@
 F 0 "J6" H 5455 4875 50  0000 L CNN
 F 1 "Conn_01x12" H 5580 4161 50  0001 L CNN
-F 2 "Adafruit_PinHeader_2.54mm:Adafruit_Feather_PinHeader_1x12_P2.54mm" H 5500 4260 50  0001 C CNN
+F 2 "Adafruit:Adafruit_Feather_PinHeader_1x12_P2.54mm" H 5500 4260 50  0001 C CNN
 F 3 "~" H 5500 4260 50  0001 C CNN
 	1    5500 4260
@@
 F 0 "J7" H 6495 4710 50  0000 L CNN
 F 1 "Conn_01x16" H 6620 3796 50  0001 L CNN
-F 2 "Adafruit_PinHeader_2.54mm:Adafruit_Feather_PinHeader_1x16_P2.54mm" H 6540 3895 50  0001 C CNN
+F 2 "Adafruit:Adafruit_Feather_PinHeader_1x16_P2.54mm" H 6540 3895 50  0001 C CNN
 F 3 "~" H 6540 3895 50  0001 C CNN
 	1    6540 3895
@@
 F 0 "R6" H 9384 1806 50  0000 L CNN
 F 1 "100k" H 9384 1715 50  0000 L CNN
-F 2 "Resistor_SMD:R_0603_1608Metric" H 9325 1760 50  0001 C CNN
+F 2 "Resistor_SMD:R_0805_2012Metric" H 9325 1760 50  0001 C CNN
 F 3 "~" H 9325 1760 50  0001 C CNN
 	1    9325 1760
@@
 F 0 "R7" H 10799 1311 50  0000 L CNN
 F 1 "2k2" H 10799 1220 50  0000 L CNN
-F 2 "Resistor_SMD:R_0603_1608Metric" H 10740 1265 50  0001 C CNN
+F 2 "Resistor_SMD:R_0805_2012Metric" H 10740 1265 50  0001 C CNN
 F 3 "~" H 10740 1265 50  0001 C CNN
 	1    10740 1265
@@
 Wire Wire Line
 	10740 990  10740 1165
-Text Notes 7170 6350 0    75   ~ 0
-1) All resistors are 0603 size.\n\n2) All capacitors except for C6, C8, C9 and C10 are 0603 size.\n\n3) Capcitors C6, C8, C9 and C10 are 0805 size.\n\n4) All LEDs are 0805 size.
+Text Notes 7075 6315 0    60   ~ 0
+1) Originally, all resistors were 0603. For this project, they were all changed to 0805.\n\n2) Capacitors C5, C6, C8, C9 and C10 are 0805 size.\n\n3) Originally, capacitors C1, C2, C3, C4 and C7 were 0603 size. \nFor this project, they were all changed to 0805.\n\n4) All LEDs are 0805 size for better visibility.
 Text Notes 8940 5440 0    100  ~ 0
 Notes
@@
 F 0 "FID1" H 6380 7276 50  0000 L CNN
 F 1 "Fiducial" H 6380 7185 50  0000 L CNN
-F 2 "Fiducial:Fiducial_0.5mm_Mask1mm" H 6295 7230 50  0001 C CNN
+F 2 "Fiducial:Fiducial_1mm_Mask2mm" H 6295 7230 50  0001 C CNN
 F 3 "~" H 6295 7230 50  0001 C CNN
 	1    6295 7230
@@
 U 1 1 60E99A86
 P 5870 7230
-F 0 "H4" H 5970 7230 50  0000 L CNN
+F 0 "H4" H 5815 7355 50  0000 L CNN
 F 1 "Mounting Hole" H 5970 7185 50  0001 L CNN
-F 2 "MountingHole:MountingHole_2.5mm" H 5870 7230 50  0001 C CNN
+F 2 "Adafruit:MountingHole_2.5mm" H 5870 7230 50  0001 C CNN
 F 3 "~" H 5870 7230 50  0001 C CNN
 	1    5870 7230
@@
 U 1 1 60E99A7C
 P 5575 7280
-F 0 "H3" H 5675 7330 50  0000 L CNN
+F 0 "H3" H 5520 7455 50  0000 L CNN
 F 1 "Mounting Hole w/Pad" H 5675 7238 50  0001 L CNN
-F 2 "MountingHole:MountingHole_2.5mm_Pad" H 5575 7280 50  0001 C CNN
+F 2 "Adafruit:MountingHole_2.5mm_Pad_TopOnly" H 5575 7280 50  0001 C CNN
 F 3 "~" H 5575 7280 50  0001 C CNN
 	1    5575 7280
@@
 $EndComp
 $Comp
-L Mechanical:MountingHole_Pad H1
-U 1 1 60E99A72
-P 4985 7280
-F 0 "H1" H 5085 7329 50  0000 L CNN
-F 1 "Mounting Hole w/Pad" H 5085 7238 50  0001 L CNN
-F 2 "MountingHole:MountingHole_2.5mm_Pad" H 4985 7280 50  0001 C CNN
-F 3 "~" H 4985 7280 50  0001 C CNN
-	1    4985 7280
-	1    0    0    -1
-$EndComp
-$Comp
 L Mechanical:MountingHole H2
 U 1 1 60E99A60
 P 5280 7230
-F 0 "H2" H 5380 7230 50  0000 L CNN
+F 0 "H2" H 5225 7355 50  0000 L CNN
 F 1 "Mounting Hole" H 5380 7185 50  0001 L CNN
-F 2 "MountingHole:MountingHole_2.5mm" H 5280 7230 50  0001 C CNN
+F 2 "Adafruit:MountingHole_2.5mm" H 5280 7230 50  0001 C CNN
 F 3 "~" H 5280 7230 50  0001 C CNN
 	1    5280 7230
 	1    0    0    -1
 $EndComp
-Text Notes 5155 7100 0    50   ~ 0
+Text Notes 5130 7565 0    50   ~ 0
 4 X M2.5 Screws
 $Bitmap
@@
 EndData
 $EndBitmap
+$Comp
+L Mechanical:MountingHole_Pad H1
+U 1 1 60E99A72
+P 4985 7280
+F 0 "H1" H 4930 7455 50  0000 L CNN
+F 1 "Mounting Hole w/Pad" H 5085 7238 50  0001 L CNN
+F 2 "Adafruit:MountingHole_2.5mm_Pad_TopOnly" H 4985 7280 50  0001 C CNN
+F 3 "~" H 4985 7280 50  0001 C CNN
+	1    4985 7280
+	1    0    0    -1
+$EndComp
 $EndSCHEMATC

Commit message: Se corrigen las observaciones realizadas por el docente. Adicionalmente se sube el ruteo de la placa.
Parts:
- J1: value 10118192 -> MicroUSB; Manf# (none) -> 10118192-0001LF
- J2: Manf# (none) -> S2B-PH-SM4-TB
- J4: value U.FL-R-SMT-1 -> U.FL; Manf# (none) -> U.FL-R-SMT-1(10)
- SW1: Manf# (none) -> KMR211GLFS
- U1: value ATSAMD21G18A-M -> ATSAMD21G18A; Manf# (none) -> ATSAMD21G18A-MUT
- U2: Manf# (none) -> AP2112K-3.3TRG1
- U3: value MCP73831T-2ACI/OT -> MCP73831T; Manf# (none) -> MCP73831T-2ACI/OT
- U4: value RFM95W-915S2 -> RFM95W; Manf# (none) -> RFM95W-915S2
- Y1: Manf# (none) -> ABS07AIG-32.768KHZ-D-T
Connections:
- net D2: no longer names the net of U1.23 (PA14)
- net D7: no longer names the net of U1.30 (PA21)
Changed lines of the file:
@@
 encoding utf-8
 Sheet 1 1
-Title "Adafruit Feather M0 with LoRa Radio Module"
+Title "Adafruit Feather M0 with LoRa Radio Module Adaptation"
 Date "2021-06-26"
 Rev "A"
@@
 F 2 "Crystal:Crystal_SMD_3215-2Pin_3.2x1.5mm" H 1175 3965 50  0001 C CNN
 F 3 "https://abracon.com/datasheets/ABS07AIG.pdf" H 1175 3965 50  0001 C CNN
+F 4 "ABS07AIG-32.768KHZ-D-T" H 1175 3965 50  0001 C CNN "Manf#"
 	1    1175 3965
 	1    0    0    -1
@@
 F 2 "Button_Switch_SMD:SW_Push_1P1T_NO_CK_KMR2" H 5600 5840 50  0001 C CNN
 F 3 "https://www.ckswitches.com/media/1479/kmr2.pdf" H 5600 5840 50  0001 C CNN
+F 4 "KMR211GLFS" H 5600 5840 50  0001 C CNN "Manf#"
 	1    5600 5840
 	1    0    0    -1
@@
 F 2 "Package_TO_SOT_SMD:SOT-23-5" H 1990 1775 50  0001 C CNN
 F 3 "https://www.diodes.com/assets/Datasheets/AP2112.pdf" H 1990 1550 50  0001 C CNN
+F 4 "AP2112K-3.3TRG1" H 1990 1450 50  0001 C CNN "Manf#"
 	1    1990 1450
 	1    0    0    -1
@@
 P 4300 1335
 F 0 "J1" H 4140 1690 50  0000 C CNN
-F 1 "10118192" H 4525 980 50  0000 C CNN
+F 1 "MicroUSB" H 4525 980 50  0000 C CNN
 F 2 "Connector_USB:USB_Micro-B_Amphenol_10103594-0001LF_Horizontal" H 4450 1285 50  0001 C CNN
 F 3 "https://cdn.amphenol-icc.com/media/wysiwyg/files/drawing/10118192.pdf" H 4450 1285 50  0001 C CNN
+F 4 "10118192-0001LF" H 4300 1335 50  0001 C CNN "Manf#"
 	1    4300 1335
 	1    0    0    -1
@@
 F 2 "Connector_JST:JST_PH_S2B-PH-SM4-TB_1x02-1MP_P2.00mm_Horizontal" H 5695 1335 50  0001 C CNN
 F 3 "https://www.jst-mfg.com/product/pdf/eng/ePH.pdf" H 5695 1335 50  0001 C CNN
+F 4 "S2B-PH-SM4-TB" H 5695 1335 50  0001 C CNN "Manf#"
 	1    5695 1335
 	1    0    0    -1
@@
 P 7575 1475
 F 0 "U3" H 7315 1735 50  0000 C CNN
-F 1 "MCP73831T-2ACI/OT" H 7575 1145 50  0000 C CNN
+F 1 "MCP73831T" H 7575 1145 50  0000 C CNN
 F 2 "Package_TO_SOT_SMD:SOT-23-5" H 7625 1225 50  0001 L CIN
 F 3 "http://ww1.microchip.com/downloads/en/DeviceDoc/20001984g.pdf" H 7425 1425 50  0001 C CNN
+F 4 "MCP73831T-2ACI/OT" H 7575 1475 50  0001 C CNN "Manf#"
 	1    7575 1475
 	1    0    0    -1
@@
 P 3070 5250
 F 0 "U1" H 2510 7120 50  0000 C CNN
-F 1 "ATSAMD21G18A-M" H 3170 5250 50  0000 C CNN
+F 1 "ATSAMD21G18A" H 3170 5250 50  0000 C CNN
 F 2 "Package_DFN_QFN:QFN-48-1EP_7x7mm_P0.5mm_EP5.15x5.15mm" H 4470 3400 50  0001 C CNN
 F 3 "http://ww1.microchip.com/downloads/en/DeviceDoc/SAM_D21_DA1_Family_Data%20Sheet_DS40001882E.pdf" H 3070 6250 50  0001 C CNN
+F 4 "ATSAMD21G18A-MUT" H 3070 5250 50  0001 C CNN "Manf#"
 	1    3070 5250
 	1    0    0    -1
@@
 P 8445 3965
 F 0 "U4" H 8090 4440 50  0000 C CNN
-F 1 "RFM95W-915S2" H 8930 3395 50  0000 C CNN
+F 1 "RFM95W" H 8730 3395 50  0000 C CNN
 F 2 "RF_Module:HOPERF_RFM9XW_SMD" H 5145 5615 50  0001 C CNN
 F 3 "https://www.hoperf.com/data/upload/portal/20181127/5bfcbea20e9ef.pdf" H 5145 5615 50  0001 C CNN
+F 4 "RFM95W-915S2" H 8445 3965 50  0001 C CNN "Manf#"
 	1    8445 3965
 	1    0    0    -1
@@
 P 10245 3665
 F 0 "J4" H 10195 3800 50  0000 L CNN
-F 1 "U.FL-R-SMT-1" H 10340 3665 50  0000 L CNN
+F 1 "U.FL" H 10340 3665 50  0000 L CNN
 F 2 "Connector_Coaxial:U.FL_Hirose_U.FL-R-SMT-1_Vertical" H 10245 3665 50  0001 C CNN
 F 3 "https://www.hirose.com/product/document?clcode=CL0311-0300-2-40&productname=HRMP-U.FLJ(40)&series=U.FL&documenttype=Catalog&lang=en&documentid=D31697_en" H 10245 3665 50  0001 C CNN
+F 4 "U.FL-R-SMT-1(10)" H 10245 3665 50  0001 C CNN "Manf#"
 	1    10245 3665
 	1    0    0    -1
@@
 MISO
 NoConn ~ 2000 4950
-Text Label 2050 5050 0    50   ~ 0
-D2
 Text Label 2000 5150 0    50   ~ 0
 D5
@@
 Text Label 2000 5650 0    50   ~ 0
 D6
-Text Label 2050 5750 0    50   ~ 0
-D7
 Text Label 2000 5850 0    50   ~ 0
 SDA

Commit message: Últimos retoques en el PCB de acuerdo a las correcciones realizadas.
Parts:
- added FID2: Fiducial, Fiducial:Fiducial_1mm_Mask2mm, symbol Mechanical:Fiducial
Other:
- moved on the sheet: FID1
